File: schematics/schematics_v2/ir_remote_v2.brd (EAGLE design)
At the start: 100 x 80 mm, 25 parts, among them IC1 AP1117E50G, T11 TASTER3301, T12 TASTER3301, T13 TASTER3301, T14 TASTER3301, T15 TASTER3301

Commit message: Clean up files in schematics v2
Parts:
- removed C11, C30: 18p, rcl:C0805
- removed Q4: (no value), crystal:HC49U-V
- added C63, C66: 22p, rcl:C0603_WE
- added Q5: 10MHz, Bernd:QUARZ_HC5032/2
- moved C68 168.2 mm to (61.0, 26.7), turned to 90 degrees
- moved C86 167.1 mm to (62.2, 35.6)
- moved T14 160.7 mm to (45.7, 10.2)
- moved R43 143.0 mm to (50.8, 24.1)
- moved T13 137.4 mm to (34.3, 10.2)
- moved R32 128.8 mm to (24.1, 35.6), turned to 90 degrees
- moved R31 126.8 mm to (31.8, 35.6), turned to 90 degrees
- moved IC1 121.7 mm to (14.0, 35.6)
- moved T12 116.6 mm to (24.1, 10.2)
- moved R30 116.0 mm to (27.9, 35.6), turned to 90 degrees
- moved R44 115.7 mm to (25.4, 43.2)
- moved ICD3 115.6 mm to (92.7, 24.1), turned to 90 degrees
- moved T15 115.0 mm to (57.1, 10.2)
- moved LED1 113.2 mm to (3.81, 47.0), turned to 270 degrees
- moved R29 112.3 mm to (20.3, 24.1), turned to 90 degrees
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Connections:
- removed net N$25: C11.1, IC8.31, Q4.1
- removed net N$9: C30.1, IC8.30, Q4.2
- new net N$47: C66.2, IC8.30, Q5.1
- new net N$48: C63.2, IC8.31, Q5.2
- net GND: now also C63.1, C66.1; no longer C11.2, C30.2
Routing:
- net GND: track 0.00 -> 212.4 mm, vias 0 -> 6
- net VCC: track 0.00 -> 111.7 mm, vias 0 -> 4
- net +9V: track 0.00 -> 67.2 mm, vias 0 -> 6
- net RB1: track 0.00 -> 54.9 mm, vias 0 -> 2
- net RB2: track 0.00 -> 49.6 mm, vias 0 -> 4
- net RB0: track 0.00 -> 49.2 mm, vias 0 -> 2
- net RB4: track 0.00 -> 48.1 mm, vias 0 -> 2
- net MCLR: track 0.00 -> 47.8 mm, vias 0 -> 4
- net RB7: track 0.00 -> 47.4 mm, vias 0 -> 2
- net RB6: track 0.00 -> 45.4 mm
- net N$24: track 0.00 -> 38.8 mm, vias 0 -> 2
- net RB3: track 0.00 -> 32.7 mm, vias 0 -> 5
- net N$19: track 0.00 -> 31.0 mm
- net N$48: track 0.00 -> 11.6 mm
- net N$47: track 0.00 -> 9.71 mm
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