File: schematics/schematics_v3/ir_remote_v3.brd (EAGLE design)
At the start: 100 x 80 mm, 26 parts, among them IC1 AP1117E50G, Q1 10MHz, T11 TASTER3301, T12 TASTER3301, T13 TASTER3301, T14 TASTER3301, T15 TASTER3301

Commit message: Update circuit layout
Parts:
- moved G1 2.54 mm to (74.9, 29.2)
- moved C5 1.27 mm to (58.4, 34.3)
- moved C6 1.27 mm to (58.4, 36.8)
- moved JP1 1.27 mm to (45.7, 22.9)
- moved R7 1.27 mm to (50.8, 19.1)
- moved R8 1.27 mm to (48.3, 19.1)
- moved C1 1.27 mm to (66.0, 29.2)
- moved C2 1.27 mm to (68.6, 29.2)
- moved IC8 1.27 mm to (47.0, 33.0)
- moved Q1 1.27 mm to (55.9, 35.6)

Commit message: Add files via upload
IR-Remote Layout
Parts:
- moved IC1 13.7 mm to (71.1, 36.8), turned to 0 degrees
- moved C7 11.5 mm to (48.3, 20.3), turned to 180 degrees
- moved G1 9.67 mm to (71.1, 20.3), turned to 270 degrees
- moved R1 6.48 mm to (34.3, 39.4), turned to 0 degrees
- moved JP1 6.48 mm to (47.0, 16.5)
- moved R8 6.35 mm to (53.3, 22.9), turned to 0 degrees
- moved C5 5.68 mm to (63.5, 31.8), turned to 180 degrees
- moved C6 5.68 mm to (63.5, 34.3), turned to 180 degrees
- moved R2 5.24 mm to (34.3, 35.6), turned to 0 degrees
- moved C1 5.08 mm to (71.1, 29.2), turned to 180 degrees
- moved R3 4.02 mm to (34.3, 31.8), turned to 0 degrees
- moved C3 4.02 mm to (55.9, 25.4)
- moved C2 3.59 mm to (71.1, 26.7), turned to 180 degrees
- moved Q1 3.59 mm to (58.4, 33.0)
- moved R7 2.84 mm to (53.3, 20.3), turned to 0 degrees
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Routing:
- net GND: track 0.00 -> 101.0 mm, vias 0 -> 3
- net VCC: track 0.00 -> 23.6 mm
- net RB4: track 0.00 -> 21.9 mm
- net N$47: track 0.00 -> 13.5 mm
- net RB6: track 0.00 -> 12.5 mm, vias 0 -> 1
- net RB7: track 0.00 -> 11.8 mm, vias 0 -> 1
- net N$48: track 0.00 -> 10.4 mm
- net +9V: track 0.00 -> 9.63 mm, vias 0 -> 1
- net RB2: track 0.00 -> 7.49 mm
- net RB3: track 0.00 -> 6.40 mm
- net MCLR: track 0.00 -> 2.62 mm
- net N$24: track 0.00 -> 0.64 mm
