File: schematics/schematics_v4/ir_remote_v4.brd (EAGLE design)
At the start: 78.4 x 49.5 mm, 26 parts, among them IC1 AP1117E50G, Q1 10MHz, T11 TASTER3301, T12 TASTER3301, T13 TASTER3301, T14 TASTER3301, T15 TASTER3301

Commit message: Improve schematics v4
Routing:
- net VCC: track 85.7 -> 95.3 mm
- net RB2: track 38.7 -> 45.9 mm
- net RB1: track 36.8 -> 43.5 mm
- net RB0: track 33.9 -> 39.5 mm
- net RB3: track 28.0 -> 32.3 mm
Changed lines of the file:
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@@
 <setting verticaltext="up"/>
 </settings>
-<grid distance="0.3175" unitdist="mm" unit="mm" style="lines" multiple="1" display="yes" altdistance="2.5" altunitdist="mil" altunit="mil"/>
+<grid distance="0.15875" unitdist="mm" unit="mm" style="lines" multiple="1" display="yes" altdistance="2.5" altunitdist="mil" altunit="mil"/>
 <layers>
 <layer number="1" name="Top" color="4" fill="1" visible="yes" active="yes"/>
@@
 <wire x1="51.7525" y1="31.4325" x2="48.26" y2="34.925" width="1.27" layer="16"/>
 <wire x1="48.26" y1="34.925" x2="37.7825" y2="34.925" width="1.27" layer="16"/>
+<wire x1="56.1975" y1="31.4325" x2="59.3725" y2="34.6455" width="0" layer="19" extent="1-1"/>
 <via x="37.7825" y="34.925" extent="1-16" drill="0.6" shape="octagon"/>
-<wire x1="56.1975" y1="31.4325" x2="59.3725" y2="34.6455" width="0" layer="19" extent="1-1"/>
 </signal>
 <signal name="GND">
@@
 <wire x1="23.1775" y1="30.48" x2="28.575" y2="30.48" width="0.4064" layer="16"/>
 <wire x1="28.575" y1="30.48" x2="31.4325" y2="33.3375" width="0.4064" layer="16"/>
-<wire x1="31.4325" y1="33.3375" x2="37.465" y2="33.3375" width="0.4064" layer="16"/>
+<wire x1="31.4325" y1="33.3375" x2="37.465" y2="33.3375" width="1.27" layer="16"/>
 <wire x1="24.0538" y1="45.1612" x2="23.1394" y2="45.1612" width="0.4064" layer="16"/>
 </signal>
@@
 <wire x1="38.1" y1="33.02" x2="37.7825" y2="33.3375" width="1.27" layer="16"/>
 <via x="37.7825" y="33.3375" extent="1-16" drill="0.6" shape="octagon"/>
+<wire x1="33.655" y1="32.385" x2="33.655" y2="33.3375" width="0.4064" layer="16"/>
 <wire x1="54.61" y1="29.845" x2="54.61" y2="24.4475" width="0" layer="19" extent="1-1"/>
-<wire x1="37.7825" y1="33.3375" x2="38.735" y2="33.3375" width="0" layer="19" extent="1-16"/>
-<wire x1="38.735" y1="33.3375" x2="40.005" y2="32.0675" width="0" layer="19" extent="1-16"/>
-<wire x1="40.005" y1="32.0675" x2="33.655" y2="32.385" width="0" layer="19" extent="1-16"/>
+<wire x1="37.7825" y1="33.3375" x2="38.57625" y2="33.3375" width="0.4064" layer="1"/>
+<wire x1="38.57625" y1="33.3375" x2="39.6875" y2="32.22625" width="0.4064" layer="1"/>
+<wire x1="39.6875" y1="32.22625" x2="41.275" y2="32.22625" width="0.4064" layer="1"/>
+<wire x1="41.275" y1="32.22625" x2="33.655" y2="32.385" width="0" layer="19" extent="1-16"/>
+<wire x1="38.57625" y1="34.925" x2="39.52875" y2="33.9725" width="0.4064" layer="1"/>
+<wire x1="37.7825" y1="34.925" x2="38.57625" y2="34.925" width="0.4064" layer="1"/>
+<wire x1="40.16375" y1="33.02" x2="41.43375" y2="33.02" width="0.4064" layer="1"/>
+<wire x1="39.52875" y1="33.49625" x2="39.52875" y2="33.9725" width="0.4064" layer="1"/>
+<wire x1="39.52875" y1="33.49625" x2="40.16375" y2="33.02" width="0.4064" layer="1"/>
 </signal>
 <signal name="D0_LCD">
@@
 <contactref element="IC8" pad="9"/>
 <wire x1="36.195" y1="39.0525" x2="35.56" y2="39.6875" width="0.4064" layer="1"/>
-<wire x1="36.195" y1="33.3375" x2="36.195" y2="39.0525" width="0.4064" layer="1"/>
+<wire x1="36.195" y1="32.385" x2="36.195" y2="39.0525" width="0.4064" layer="1"/>
 <wire x1="35.56" y1="39.6875" x2="33.97" y2="39.6875" width="0.4064" layer="1"/>
 <wire x1="27.6606" y1="45.1612" x2="28.8163" y2="45.1612" width="0.4064" layer="16"/>
@@
 <wire x1="50.165" y1="40.9575" x2="50.19" y2="40.9325" width="0.4064" layer="1"/>
 <wire x1="50.19" y1="40.9325" x2="50.19" y2="38.82" width="0.4064" layer="1"/>
-<wire x1="36.195" y1="33.3375" x2="41.19" y2="30.62" width="0" layer="19" extent="1-1"/>
+<wire x1="36.195" y1="32.385" x2="37.94125" y2="30.63875" width="0.4064" layer="1"/>
+<wire x1="37.94125" y1="30.63875" x2="41.17125" y2="30.63875" width="0.4064" layer="1"/>
+<wire x1="41.17125" y1="30.63875" x2="41.19" y2="30.62" width="0.4064" layer="1"/>
 </signal>
 <signal name="RB2">
@@
 <contactref element="IC8" pad="32"/>
 <contactref element="IC8" pad="10"/>
-<wire x1="35.56" y1="33.02" x2="35.56" y2="33.9725" width="0.4064" layer="1"/>
-<wire x1="35.56" y1="33.9725" x2="34.925" y2="34.925" width="0.4064" layer="1"/>
-<wire x1="34.925" y1="34.925" x2="33.97" y2="34.925" width="0.4064" layer="1"/>
 <wire x1="27.6606" y1="32.4612" x2="27.6606" y2="34.6456" width="0.4064" layer="16"/>
 <wire x1="27.6606" y1="34.6456" x2="29.845" y2="36.83" width="0.4064" layer="16"/>
@@
 <wire x1="51.435" y1="36.83" x2="53.0225" y2="38.4175" width="0.4064" layer="16"/>
 <wire x1="53.0225" y1="38.4175" x2="54.2925" y2="38.4175" width="0.4064" layer="16"/>
-<wire x1="35.56" y1="33.02" x2="41.19" y2="29.82" width="0" layer="19" extent="1-1"/>
+<wire x1="33.97" y1="34.925" x2="33.97" y2="33.6575" width="0.4064" layer="1"/>
+<wire x1="33.97" y1="33.6575" x2="34.6075" y2="33.02" width="0.4064" layer="1"/>
+<wire x1="34.6075" y1="33.02" x2="34.6075" y2="32.7025" width="0.4064" layer="1"/>
+<wire x1="34.6075" y1="32.7025" x2="37.465" y2="29.845" width="0.4064" layer="1"/>
+<wire x1="37.465" y1="29.845" x2="41.165" y2="29.845" width="0.4064" layer="1"/>
+<wire x1="41.165" y1="29.845" x2="41.19" y2="29.82" width="0.4064" layer="1"/>
 </signal>
 <signal name="RB3">
@@
 <contactref element="R4" pad="2"/>
 <contactref element="IC8" pad="11"/>
-<wire x1="37.1475" y1="30.48" x2="33.97" y2="30.48" width="0.4064" layer="1"/>
 <via x="33.9725" y="28.575" extent="1-16" drill="0.6" shape="octagon"/>
 <wire x1="33.9725" y1="28.575" x2="33.97" y2="28.5775" width="0.4064" layer="1"/>
@@
 <wire x1="17.4625" y1="19.7993" x2="17.5006" y2="19.7612" width="0.4064" layer="16"/>
 <wire x1="18.415" y1="22.5425" x2="27.6225" y2="22.5425" width="0.4064" layer="16"/>
-<wire x1="37.1475" y1="30.48" x2="41.19" y2="29.02" width="0" layer="19" extent="1-1"/>
+<wire x1="33.97" y1="28.5775" x2="39.055" y2="28.5775" width="0.4064" layer="1"/>
+<wire x1="39.055" y1="28.5775" x2="39.52875" y2="29.05125" width="0.4064" layer="1"/>
+<wire x1="39.52875" y1="29.05125" x2="41.15875" y2="29.05125" width="0.4064" layer="1"/>
+<wire x1="41.15875" y1="29.05125" x2="41.19" y2="29.02" width="0.4064" layer="1"/>
 </signal>
 <signal name="RB4">
@@
 <contactref element="T11" pad="1"/>
 <contactref element="R1" pad="2"/>
-<wire x1="36.83" y1="33.655" x2="36.83" y2="44.1325" width="0.4064" layer="1"/>
+<wire x1="36.83" y1="33.02" x2="36.83" y2="44.1325" width="0.4064" layer="1"/>
 <wire x1="36.83" y1="44.1325" x2="36.195" y2="44.7675" width="0.4064" layer="1"/>
 <wire x1="36.195" y1="44.7675" x2="33.97" y2="44.7675" width="0.4064" layer="1"/>
@@
 <wire x1="17.4625" y1="46.6725" x2="18.0975" y2="47.3075" width="0.4064" layer="16"/>
 <wire x1="18.0975" y1="47.3075" x2="20.0025" y2="47.3075" width="0.4064" layer="16"/>
-<wire x1="36.83" y1="33.655" x2="41.19" y2="31.42" width="0" layer="19" extent="1-1"/>
+<wire x1="36.83" y1="33.02" x2="38.4175" y2="31.4325" width="0.4064" layer="1"/>
+<wire x1="38.4175" y1="31.4325" x2="41.1775" y2="31.4325" width="0.4064" layer="1"/>
+<wire x1="41.1775" y1="31.4325" x2="41.19" y2="31.42" width="0.4064" layer="1"/>
 </signal>
 <signal name="RD0_LED">
