File: schematics/schematics_v5_3/ir_remote_v3.brd (EAGLE design)
At the start: 73.8 x 39.2 mm, 27 parts, among them IC1 AP1117E50G, Q1 10MHz, T11 TASTER3301, T12 TASTER3301, T13 TASTER3301, T14 TASTER3301, T15 TASTER3301

Commit message: Add pwm
Parts:
- removed IC1: AP1117E50G, Bernd_110428:SOT223
- added IC3: LM2937IMP-5.0_NOPB, LM2937IMP-5.0_NOPB:SOT230P700X180-4N
- moved G1 16.3 mm to (63.8, 28.4), turned to 90 degrees
- moved C3 3.37 mm to (61.9, 20.0), turned to 90 degrees
- moved C2 3.37 mm to (66.4, 20.0), turned to 90 degrees
- moved C1 1.21 mm to (68.6, 20.0), turned to 90 degrees
Connections:
- net +9V: now also IC3.1; no longer IC1.3
- net GND: now also IC3.2, IC3.4; no longer IC1.1
- net VCC: now also IC3.3; no longer IC1.2, IC1.4
Routing:
- net VCC: track 106.8 -> 97.5 mm, vias 4 -> 3
- net GND: track 191.4 -> 196.9 mm, vias 3 -> 1
- net +9V: track 18.3 -> 22.3 mm, vias 0 -> 2
- added copper zone on layer 1, net GND
- removed copper zone on layer 1, net VCC
